Commit message: update

File: robot_urdf/urdf/robot4.xacro (robot description, xacro)
@@ -138,5 +138,5 @@
   </link>
   <joint name="camera_joint" type="fixed">
-	    <axis xyz="0 1 0" />
+		<axis xyz="0 0 1" />
 	    <origin xyz="0.23 0 0.0" rpy="0 0 0"/>
 	    <parent link="link_chassis"/>

Commit message: fix camera location and cleaning up the repo

File: robot_urdf/urdf/robot4.xacro (robot description, xacro)
@@ -115,31 +115,92 @@
     <joint_properties damping="1.0" friction="1.0"/>
   </joint>
+  <!-- New link for camera mount -->
+  <link name="camera_mount">
+    <inertial>
+      <mass value="0.1"/>
+      <origin xyz="0 0 0" rpy="0 0 0"/>
+      <inertia ixx="0.0001" ixy="0.0" ixz="0.0" iyy="0.0001" iyz="0.0" izz="0.0001"/>
+    </inertial>
+    <visual>
+      <origin xyz="0 0 0" rpy="0 0 0"/>
+      <geometry>
+        <box size="0.1 0.1 0.1"/>
+      </geometry>
+      <material>
+        <color rgba="0.5 0.5 0.5 1.0"/>
+      </material>
+    </visual>
+    <collision>
+      <origin xyz="0 0 0" rpy="0 0 0"/>
+      <geometry>
+        <box size="0.1 0.1 0.1"/>
+      </geometry>
+    </collision>
+  </link>
+  <!-- Joint to connect camera mount to chassis -->
+  <joint name="camera_mount_joint" type="fixed">
+    <parent link="link_chassis"/>
+    <child link="camera_mount"/>
+    <origin xyz="0 0 0.1" rpy="0 0 0"/>
+  </joint>
+  <!-- Adjust the camera link to be a child of the camera mount -->
+  <joint name="camera_joint" type="continuous">
+    <command_interface name="velocity">
+      <!-- <param name='min'> ${rotating_limlow} </param>
+      <param name='max'> ${rotating_limhigh} </param> -->
+    </command_interface>
+    <state_interface name="position"/>
+    <state_interface name="velocity"/>
+    <state_interface name="effort"/>
+    <axis xyz="0 0 1" />
+    <origin xyz="0 0 0.1" rpy="0 0 0"/>
+    <parent link="camera_mount"/>
+    <child link="camera_link"/>
+  </joint>
   <link name="camera_link">
-	    <collision>
-	      <origin xyz="0 0 0.025" rpy="0 0 0"/>
-	      <geometry>
-		<box size="0.05 0.05 0.05"/>
-	      </geometry>
-	    </collision>
-	    <visual>
-	      <origin xyz="0 0 0.025" rpy="0 0 0"/>
-	      <geometry>
-		<box size="0.05 0.05 0.05"/>
-	      </geometry>
-	      <material name="red">
-		<color rgba="1 0 0 1"/>
-	      </material>
-	    </visual>
-	    <inertial>
-	      <mass value="1e-5" />
-	      <origin xyz="0 0 0" rpy="0 0 0"/>
-	      <inertia ixx="1e-6" ixy="0" ixz="0" iyy="1e-6" iyz="0" izz="1e-6" />
-	    </inertial>
-  </link>
-  <joint name="camera_joint" type="fixed">
-		<axis xyz="0 0 1" />
-	    <origin xyz="0.23 0 0.0" rpy="0 0 0"/>
-	    <parent link="link_chassis"/>
-	    <child link="camera_link"/>
-	 </joint>
+    <collision>
+      <origin xyz="0 0 0.25" rpy="0 0 0"/>
+      <geometry>
+        <box size="0.05 0.05 0.05"/>
+      </geometry>
+    </collision>
+    <visual>
+      <origin xyz="0 0 0.1" rpy="0 0 0"/>
+      <geometry>
+        <box size="0.05 0.05 0.1"/>
+      </geometry>
+      <material name="red">
+        <color rgba="1 0 0 1"/>
+      </material>
+    </visual>
+    <inertial>
+      <mass value="1e-5" />
+      <origin xyz="0 0 0" rpy="0 0 0"/>
+      <inertia ixx="1e-6" ixy="0" ixz="0" iyy="1e-6" iyz="0" izz="1e-6" />
+    </inertial>
+  </link>
+  <transmission name="camera_trans">
+    <type>transmission_interface/SimpleTransmission</type>
+    <joint name="camera_joint">
+      <hardwareInterface>hardware_interface/VelocityJointInterface</hardwareInterface>
+    </joint>
+    <actuator name="camera_motor">
+      <mechanicalReduction>m1</mechanicalReduction>
+    </actuator>
+  </transmission>
+  <!-- ros2_control tag -->
+  <ros2_control name="my_robot_control" type="system">
+    <hardware>
+      <plugin>gazebo_ros2_control/GazeboSystem</plugin>
+    </hardware>
+    <joint name="camera_joint">
+      <command_interface name="velocity">
+        <param name="min">-10</param>
+        <param name="max">10</param>
+      </command_interface>
+      <state_interface name="position"/>
+      <state_interface name="velocity"/>
+      <state_interface name="effort"/>
+    </joint>
+  </ros2_control>
 </robot>
